File: hardware/lochord.kicad_sch (KiCad schematic)
At the start: 0 parts

Commit message: hw: added esp32 footprint
Parts:
- added U1: ESP32-S3-WROOM-1, RF_Module:ESP32-S3-WROOM-1, symbol RF_Module:ESP32-S3-WROOM-1
Connections:
- new net: U1.1 (GND), U1.40 (GND), U1.41 (GND)
Other:
- title: (none) -> LoChord
Changed lines of the file:
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@@
 	(generator_version "10.0")
 	(paper "A4")
+	(title_block
+		(title "LoChord")
+		(date "2026-05-08")
+		(rev "v1")
+	)
+	(symbol
+		(lib_id "RF_Module:ESP32-S3-WROOM-1")
+		(at 173.99 58.42 0)
+		(unit 1)
+		(body_style 1)
+		(exclude_from_sim no)
+		(in_bom yes)
+		(on_board yes)
+		(in_pos_files yes)
+		(dnp no)
+		(fields_autoplaced yes)
+		(property "Reference" "U1"
+			(at 176.1333 27.94 0)
+			(show_name no)
+			(do_not_autoplace no)
+			(effects
+				(font
+					(size 1.27 1.27)
+				)
+				(justify left)
+			)
+		)
+		(property "Value" "ESP32-S3-WROOM-1"
+			(at 176.1333 30.48 0)
+			(show_name no)
+			(do_not_autoplace no)
+			(effects
+				(font
+					(size 1.27 1.27)
+				)
+				(justify left)
+			)
+		)
+		(property "Footprint" "RF_Module:ESP32-S3-WROOM-1"
+			(at 173.99 55.88 0)
+			(hide yes)
+			(show_name no)
+			(do_not_autoplace no)
+			(effects
+				(font
+					(size 1.27 1.27)
+				)
+			)
+		)
+		(property "Datasheet" "https://www.espressif.com/sites/default/files/documentation/esp32-s3-wroom-1_wroom-1u_datasheet_en.pdf"
+			(at 173.99 58.42 0)
+			(hide yes)
+			(show_name no)
+			(do_not_autoplace no)
+			(effects
+				(font
+					(size 1.27 1.27)
+				)
+			)
+		)
+		(property "Description" "RF Module, ESP32-S3 SoC, Wi-Fi 802.11b/g/n, Bluetooth, BLE, 32-bit, 3.3V, onboard antenna, SMD"
+			(at 173.99 58.42 0)
+			(hide yes)
+			(show_name no)
+			(do_not_autoplace no)
+			(effects
+				(font
+					(size 1.27 1.27)
+				)
+			)
+		)
+		(pin "26"
+		)
+		(pin "25"
+		)
+		(pin "31"
+		)
+		(pin "18"
+		)
+		(pin "29"
+		)
+		(pin "21"
+		)
+		(pin "19"
+		)
+		(pin "35"
+		)
+		(pin "16"
+		)
+		(pin "15"
+		)
+		(pin "14"
+		)
+		(pin "13"
+		)
+		(pin "12"
+		)
+		(pin "11"
+		)
+		(pin "10"
+		)
+		(pin "9"
+		)
+		(pin "36"
+		)
+		(pin "38"
+		)
+		(pin "8"
+		)
+		(pin "7"
+		)
+		(pin "6"
+		)
+		(pin "5"
+		)
+		(pin "4"
+		)
+		(pin "3"
+		)
+		(pin "2"
+		)
+		(pin "1"
+		)
+		(pin "37"
+		)
+		(pin "40"
+		)
+		(pin "41"
+		)
+		(pin "20"
+		)
+		(pin "39"
+		)
+		(pin "23"
+		)
+		(pin "24"
+		)
+		(pin "17"
+		)
+		(pin "33"
+		)
+		(pin "30"
+		)
+		(pin "27"
+		)
+		(pin "28"
+		)
+		(pin "32"
+		)
+		(pin "34"
+		)
+		(pin "22"
+		)
+		(instances
+			(project "lochord"
+				(path "/c3bb49aa-b062-4b61-997a-34eb2bc951f1"
+					(reference "U1")
+					(unit 1)
+				)
+			)
+		)
+	)
 	(sheet_instances
 		(path "/"
