File: lochord_hw/lochord_hw.kicad_sch (KiCad schematic)
At the start: 23 parts, among them J1 TYPE-C-31-M-12, SW1 TS-1088-AR02016, SW2 TS-1088-AR02016, SW3 UI_Encoder, SW4 RotaryEncoder_Mappable1, SW5 RotaryEncoder_Mappable2, U2 ESP32-S3-WROOM-1-N8R8, U3 LD1117S33TR_SOT223

Commit message: atomic14 pcb design
Parts:
- removed SW4: RotaryEncoder_Mappable1, Rotary_Encoder:RotaryEncoder_Alps_EC11E-Switch_Vertical_H20mm_CircularMountingHoles, symbol Device:RotaryEncoder_Switch
- removed SW5: RotaryEncoder_Mappable2, Rotary_Encoder:RotaryEncoder_Alps_EC11E-Switch_Vertical_H20mm_CircularMountingHoles, symbol Device:RotaryEncoder_Switch
- added R10, R11, R12, R13, R14, R9: 10K, Resistor_SMD:R_0603_1608Metric, symbol Device:R
- added SW10, SW12: SW_Push, Switch_Keyboard_Kailh:SW_Kailh_Choc_V2_1.50u, symbol Switch:SW_Push
- added SW11, SW14: SW_Push, Switch_Keyboard_Kailh:SW_Kailh_Choc_V2_1.00u, symbol Switch:SW_Push
- added SW13, SW15: UI_Encoder, Rotary_Encoder:RotaryEncoder_Alps_EC11E-Switch_Vertical_H20mm_CircularMountingHoles, symbol Device:RotaryEncoder_Switch
- added SW6, SW7, SW8, SW9: SW_Push, Switch_Keyboard_Kailh:SW_Kailh_Choc_V2_2.25u_90deg, symbol Switch:SW_Push
Connections:
- net +3V3: now also C6.2, R5.1, U2.2 (3V3), R10.1, R11.1, R12.1, R13.1, R14.1, R9.1; no longer C6.1
- net GND: now also C6.1, SW10.2, SW11.2, SW12.2, SW13.C, SW13.S2, SW14.2, SW15.C, SW15.S2, SW6.2, SW7.2, SW8.2, SW9.2
- net GPIO13: now also SW9.1
- net GPIO14: now also SW8.1
- net GPIO15: now also R8.2, SW3.B
- net GPIO16: now also R7.2, SW3.S1
- net GPIO17: now also R9.2, SW13.A
- net GPIO18: now also R10.2, SW13.B
- net GPIO21: now also R12.2, SW15.A; no longer R5.1
- net GPIO39: now also SW6.1
- net GPIO40: now also SW12.1
- net GPIO41: now also SW10.1
- net GPIO42: now also SW11.1
- net GPIO43: now also SW14.1
- net GPIO45: now also SW7.1; no longer R8.2, SW3.B
- net GPIO47: now also R13.2, SW15.B; no longer R7.2, SW3.S1
- net GPIO48: now also R14.2, SW15.S1; no longer R6.2, SW3.A
- net GPIO7: now also R6.2, SW3.A
- net GPIO8: now also R11.2, SW13.S1
Other:
- moved on the sheet: C1, C2, C3, C4, C5, C6, D3, J1, R1, R2, R3, R4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

Commit message: hw: pcb design for esp32-p4
Parts:
- removed C2: 22uF, Capacitor_SMD:C_0603_1608Metric, symbol Device:C
- removed D3: RED, LED_SMD:LED_0603_1608Metric, symbol Device:LED
- removed J1: TYPE-C-31-M-12, TYPE-C-31-M-12:HRO_TYPE-C-31-M-12, symbol TYPE-C-31-M-12:TYPE-C-31-M-12
- removed SW1, SW2: TS-1088-AR02016, easyeda2kicad:SW-SMD_L3.9-W3.0-P4.45, symbol easyeda2kicad:TS-1088-AR02016
- removed SW11, SW14: SW_Push, Switch_Keyboard_Kailh:SW_Kailh_Choc_V2_1.00u, symbol Switch:SW_Push
- removed SW12: SW_Push, Switch_Keyboard_Kailh:SW_Kailh_Choc_V2_1.50u, symbol Switch:SW_Push
- removed SW13, SW15, SW3: UI_Encoder, Rotary_Encoder:RotaryEncoder_Alps_EC11E-Switch_Vertical_H20mm_CircularMountingHoles, symbol Device:RotaryEncoder_Switch
- removed U2: ESP32-S3-WROOM-1-N8R8, PCM_Espressif:ESP32-S3-WROOM-1, symbol PCM_Espressif:ESP32-S3-WROOM-1
- removed U3: LD1117S33TR_SOT223, Package_TO_SOT_SMD:SOT-223-3_TabPin2, symbol Regulator_Linear:LD1117S33TR_SOT223
- added C10, C11, C13, C14, C16, C18, C20, C23, C26: 100nF, Capacitor_SMD:C_0402_1005Metric, symbol Device:C
- added C12, C15, C17, C19, C21, C22, C9: 10uF, Capacitor_SMD:C_0603_1608Metric, symbol Device:C
- added C2: 100uF/10V, Capacitor_SMD:CP_Elec_5x5.4, symbol Device:C_Polarized
- added C24, C25: 220uF/6.3V, Capacitor_SMD:CP_Elec_6.3x5.4, symbol Device:C_Polarized
- added C27, C28, C29, C30, C31, C32: 10nF, Capacitor_SMD:C_0402_1005Metric, symbol Device:C
- added C7, C8: 1uF, Capacitor_SMD:C_0402_1005Metric, symbol Device:C
- added D1: GREEN, LED_SMD:LED_0603_1608Metric, symbol Device:LED
- added FB1: 600R@100MHz, Inductor_SMD:L_0603_1608Metric, symbol Device:FerriteBead
- added J1: USB-C 16P, Connector_USB:USB_C_Receptacle_HRO_TYPE-C-31-M-12, symbol Connector:USB_C_Receptacle_USB2.0_16P
- added J2: DEBUG USJ, Connector_PinHeader_2.54mm:PinHeader_1x04_P2.54mm_Vertical, symbol Connector_Generic:Conn_01x04
- added J3: JOYSTICK_NS, lochord:FPC_1x05_P0.50mm_Horizontal_ZIF, symbol lochord:JOYSTICK_NS_FPC5
- added J4: LCD_NV3007, lochord:FPC_1x08_P0.50mm_Horizontal_ZIF, symbol lochord:LCD_NV3007_FPC8
- added J5: PJ-320D, Connector_Audio:Jack_3.5mm_PJ320D_Horizontal, symbol Connector_Audio:AudioJack4
- added M1: JOYSTICK_NS_MODULE, lochord:Joystick_NintendoSwitch_Module, symbol lochord:JOYSTICK_NS_MODULE
- added M2: NV3007_2.79in_428x142, lochord:Display_NV3007_2.79in_428x142, symbol lochord:NV3007_PANEL_2V79
- added Q1: SI2302, Package_TO_SOT_SMD:SOT-23, symbol Transistor_FET:2N7002
- added R15: 0R, Resistor_SMD:R_0402_1005Metric, symbol Device:R
- added R16: 100k, Resistor_SMD:R_0402_1005Metric, symbol Device:R
- added R17: 100R, Resistor_SMD:R_0402_1005Metric, symbol Device:R
- added R18, R19, R20, R21: 33R, Resistor_SMD:R_0402_1005Metric, symbol Device:R
- added R22, R23: 4.7k, Resistor_SMD:R_0402_1005Metric, symbol Device:R
- added R24: 10k, Resistor_SMD:R_0402_1005Metric, symbol Device:R
- added R25, R26: 10R, Resistor_SMD:R_0402_1005Metric, symbol Device:R
- added RE1, RE2, RE3: EC11E15244G1, Rotary_Encoder:RotaryEncoder_Alps_EC11E-Switch_Vertical_H20mm_CircularMountingHoles, symbol Device:RotaryEncoder_Switch
- added SW1: EN, lochord:SW_SMD_TS-1088-AR02016_3.9x3.0mm, symbol Switch:SW_Push
- added SW2: BOOT, lochord:SW_SMD_TS-1088-AR02016_3.9x3.0mm, symbol Switch:SW_Push
- added SW3: CHORD1, Switch_Keyboard_Kailh:SW_Kailh_Choc_V1_2.00u, symbol Switch:SW_Push
- added SW4: CHORD2, Switch_Keyboard_Kailh:SW_Kailh_Choc_V1_2.00u, symbol Switch:SW_Push
- added SW5: CHORD3, Switch_Keyboard_Kailh:SW_Kailh_Choc_V1_2.00u, symbol Switch:SW_Push
- added TP1: USB_HS_DM, TestPoint:TestPoint_Pad_D1.5mm, symbol Connector:TestPoint
- added TP2: USB_HS_DP, TestPoint:TestPoint_Pad_D1.5mm, symbol Connector:TestPoint
- added TP3: U0TXD, TestPoint:TestPoint_Pad_D1.5mm, symbol Connector:TestPoint
- added TP4: U0RXD, TestPoint:TestPoint_Pad_D1.5mm, symbol Connector:TestPoint
- added U1: WT0132P4-A1-N16R32, lochord:WT0132P4-A1, symbol lochord:WT0132P4-A1-N16R32
- added U2: AMS1117-3.3, Package_TO_SOT_SMD:SOT-223-3_TabPin2, symbol Regulator_Linear:AMS1117-3.3
- added U3: LP5907MFX-3.3, Package_TO_SOT_SMD:SOT-23-5, symbol Regulator_Linear:LP5907MFX-3.3
- added U4: USBLC6-2SC6, Package_TO_SOT_SMD:SOT-23-6, symbol Power_Protection:USBLC6-2SC6
- added U5: ES8388, lochord:QFN-28-1EP_4x4mm_P0.45mm_EP2.6x2.6mm_ThermalVias, symbol lochord:ES8388
- C1: value 10uF -> 1uF; footprint Capacitor_SMD:C_0603_1608Metric -> Capacitor_SMD:C_0402_1005Metric; LCSC C59461 -> C52923
- C3: value 100nF -> 22uF/25V; footprint Capacitor_SMD:C_0603_1608Metric -> Capacitor_SMD:C_0805_2012Metric; LCSC C14663 -> C45783
- C4, C6: footprint Capacitor_SMD:C_0603_1608Metric -> Capacitor_SMD:C_0402_1005Metric; LCSC C14663 -> C1525
- C5: value 1uF -> 22uF/25V; footprint Capacitor_SMD:C_0603_1608Metric -> Capacitor_SMD:C_0805_2012Metric; LCSC C15849 -> C45783
- R1: value 5.1K -> 10k; footprint Resistor_SMD:R_0603_1608Metric -> Resistor_SMD:R_0402_1005Metric; LCSC C23186 -> C25744
- R10, R11, R12, R13, R6, R7, R8, R9: value 10K -> 10k; footprint Resistor_SMD:R_0603_1608Metric -> Resistor_SMD:R_0402_1005Metric; LCSC C25804 -> C25744
- R14: value 10K -> 22R; footprint Resistor_SMD:R_0603_1608Metric -> Resistor_SMD:R_0402_1005Metric; LCSC C25804 -> C25092
- R2: value 5.1K -> 5.1k; footprint Resistor_SMD:R_0603_1608Metric -> Resistor_SMD:R_0402_1005Metric; LCSC C23186 -> C25905
- R3: value 10K -> 5.1k; footprint Resistor_SMD:R_0603_1608Metric -> Resistor_SMD:R_0402_1005Metric; LCSC C25804 -> C25905
- R4: value 10K -> 470R; footprint Resistor_SMD:R_0603_1608Metric -> Resistor_SMD:R_0402_1005Metric; LCSC C25804 -> C25117
- R5: value 1K -> 10k; footprint Resistor_SMD:R_0603_1608Metric -> Resistor_SMD:R_0402_1005Metric; LCSC C21190 -> C25744
- SW10: value SW_Push -> LOOP; footprint Switch_Keyboard_Kailh:SW_Kailh_Choc_V2_1.50u -> Switch_Keyboard_Kailh:SW_Kailh_Choc_V1_1.00u
- SW6: value SW_Push -> CHORD4; footprint Switch_Keyboard_Kailh:SW_Kailh_Choc_V2_2.25u_90deg -> Switch_Keyboard_Kailh:SW_Kailh_Choc_V1_2.00u
- SW7: value SW_Push -> CHORD5; footprint Switch_Keyboard_Kailh:SW_Kailh_Choc_V2_2.25u_90deg -> Switch_Keyboard_Kailh:SW_Kailh_Choc_V1_1.50u
- SW8: value SW_Push -> CHORD6; footprint Switch_Keyboard_Kailh:SW_Kailh_Choc_V2_2.25u_90deg -> Switch_Keyboard_Kailh:SW_Kailh_Choc_V1_1.00u
- SW9: value SW_Push -> CHORD7; footprint Switch_Keyboard_Kailh:SW_Kailh_Choc_V2_2.25u_90deg -> Switch_Keyboard_Kailh:SW_Kailh_Choc_V1_1.50u
Connections:
- net +3V3: now also C5.1, C6.1, R1.1, C11.1, C12.1, C13.1, C14.1, C26.1, J2.1 (Pin_1), J3.2 (VCC), J4.2 (VCC), R22.1, R23.1, U2.2 (VO), U5.2 (DVDD), U5.3 (PVDD); no longer C1.1, C3.1, C6.2, R14.1, R3.1
- net +5V: now also C3.1, C2.1, C7.1, J1.A4 (VBUS), J1.A9 (VBUS), J1.B4 (VBUS), J1.B9 (VBUS), U1.41 (VCC), U2.3 (VI), U3.1 (IN), U3.3 (EN), U4.5 (VBUS)
- net EN: now also C1.1, SW1.1, U1.70 (CHIP_PU); no longer C5.1, R3.2
- net GND: now also C6.2, R3.2, C10.2, C11.2, C12.2, C13.2, C14.2, C15.2, C16.2, C17.2, C18.2, C19.2, C2.2, C20.2, C21.2, C22.2, C23.2, C26.2, C27.2, C28.2, C29.2, C30.2, C31.2, C32.2, C7.2, C8.2, C9.2, D1.1 (K), J1.A1 (GND), J1.A12 (GND), J1.B1 (GND), J1.B12 (GND), J1.SH (SHIELD), J2.2 (Pin_2), J3.1 (GND), J4.1 (GND), J5.R2, J5.S, M1.1 (MP1), M1.2 (MP2), Q1.2 (S), R16.2, R24.2, RE1.C, RE1.S2, RE2.C, RE2.S2, RE3.C, RE3.S2, SW1.2, SW2.2, SW3.2, SW4.2, SW5.2, U1.1 (GND), U1.15 (GND), U1.18 (GND), U1.21 (GND), U1.42 (GND), U1.53 (GND), U1.64 (GND), U1.73 (GND), U1.8 (GND), U1.82 (GND), U2.1 (GND), U3.2 (GND), U4.2 (GND), U5.13 (HPGND), U5.18 (AGND), U5.29 (EP), U5.4 (DGND); no longer C6.1, R1.2
- net ENC1_A: now reaches R5.2
- net ENC1_A: now also C27.1, RE1.A, U1.36 (GPIO39)
- net USB_CC1: now reaches R2.1
- net USB_CC1: now also J1.A5 (CC1)
- net GPIO0 renamed PWR_LED
- net PWR_LED: now also D1.2 (A)
- net GPIO13 renamed KEY7
- net KEY7: now also U1.49 (GPIO50)
- net GPIO14 renamed KEY6
- net KEY6: now also U1.48 (GPIO49)
- net GPIO15 renamed ENC2_A
- net ENC2_A: now also C29.1, RE2.A, U1.24 (GPIO28)
- net GPIO16 renamed ENC1_SW
- net ENC1_SW: now also RE1.S1, U1.38 (GPIO41)
- net GPIO17 renamed ENC2_B
- net ENC2_B: now also C30.1, RE2.B, U1.25 (GPIO29)
- net GPIO18 renamed ENC2_SW
- net ENC2_SW: now also RE2.S1, U1.26 (GPIO30)
- net GPIO21 renamed ENC3_B
- net ENC3_B: now also C32.1, RE3.B, U1.28 (GPIO32)
- net GPIO39 renamed KEY4
- net KEY4: now also U1.46 (GPIO47)
- net GPIO41 renamed KEY_LOOP
- net KEY_LOOP: now also U1.50 (GPIO51)
- net GPIO45 renamed KEY5
- net KEY5: now also U1.47 (GPIO48)
- net GPIO47 renamed ENC3_SW
- net ENC3_SW: now also RE3.S1, U1.29 (GPIO33)
- net GPIO48 renamed LCD_SCLK_R
- net LCD_SCLK_R: now also J4.3 (SCL)
- net GPIO7 renamed ENC1_B
- net ENC1_B: now also C28.1, RE1.B, U1.37 (GPIO40)
- net GPIO8 renamed ENC3_A
- net ENC3_A: now also C31.1, RE3.A, U1.27 (GPIO31)
- new net +3.3VA: C10.1, C15.1, C16.1, C17.1, C18.1, C9.1, FB1.2, U5.16 (HPVDD), U5.17 (AVDD)
- new net BOOT: SW2.1, U1.31 (GPIO35/BOOT)
- new net BOOTSEL: R1.2, U1.33 (GPIO36/BOOTSEL)
- new net CODEC_ADCVREF: C21.1, U5.19 (ADCVREF)
- new net CODEC_CE: R24.1, U5.26 (CE/AD0)
- new net CODEC_VMID: C22.1, C23.1, U5.20 (VMID)
- new net CODEC_VREF: C19.1, C20.1, U5.10 (VREF)
- new net HP_L: C24.2, R25.1
- new net HP_L_AC: C24.1, U5.12 (LOUT1)
- new net HP_L_J: J5.T, R25.2
- new net HP_R: C25.2, R26.1
- new net HP_R_AC: C25.1, U5.11 (ROUT1)
- new net HP_R_J: J5.R1, R26.2
- new net I2C_SCL: R23.2, U1.72 (GPIO1), U5.28 (CCLK/SCL)
- new net I2C_SDA: R22.2, U1.71 (GPIO0), U5.27 (CDATA/SDA)
- new net I2S_BCLK: R19.1, U1.68 (GPIO14)
- new net I2S_BCLK_R: R19.2, U5.5 (SCLK)
- new net I2S_DOUT: R21.1, U1.67 (GPIO13)
- new net I2S_DOUT_R: R21.2, U5.6 (DSDIN)
- new net I2S_LRCK: R20.1, U1.69 (GPIO15)
- new net I2S_LRCK_R: R20.2, U5.7 (LRCK)
- new net I2S_MCLK: R18.1, U1.66 (GPIO12)
- new net I2S_MCLK_R: R18.2, U5.1 (MCLK)
- new net JOY_SW: J3.5 (SW), U1.76 (GPIO18)
- new net JOY_X: J3.3 (X_LR), U1.74 (GPIO16)
- new net JOY_Y: J3.4 (Y_UD), U1.75 (GPIO17)
- new net JTAG_DM: J2.3 (Pin_3), U1.19 (GPIO24/USJ_D-)
- new net JTAG_DP: J2.4 (Pin_4), U1.20 (GPIO25/USJ_D+)
- new net KEY1: SW3.1, U1.43 (GPIO44)
- new net KEY2: SW4.1, U1.44 (GPIO45)
- new net KEY3: SW5.1, U1.45 (GPIO46)
- new net LCD_BL: R15.1, R17.1, U1.59 (GPIO6)
- new net LCD_BLK: J4.8 (BLK), Q1.3 (D), R15.2, R16.1
- new net LCD_BL_G: Q1.1 (G), R17.2
- new net LCD_CS: J4.7 (CS), U1.60 (GPIO7)
- new net LCD_DC: J4.6 (DC), U1.63 (GPIO10)
- new net LCD_MOSI: J4.4 (SDA), U1.61 (GPIO8)
- new net LCD_RST: J4.5 (RES), U1.65 (GPIO11)
- new net LCD_SCLK: R14.1, U1.62 (GPIO9)
- new net U0RXD: TP4.1, U1.35 (GPIO38/U0RXD)
- new net U0TXD: TP3.1, U1.34 (GPIO37/U0TXD)
- new net USB_CC2: J1.B5 (CC2), R3.1
- new net USB_DM: J1.A7 (D-), J1.B7 (D-), U1.22 (GPIO26/USB_D-), U4.1 (I/O1), U4.6 (I/O1)
- new net USB_DP: J1.A6 (D+), J1.B6 (D+), U1.23 (GPIO27/USB_D+), U4.3 (I/O2), U4.4 (I/O2)
- new net USB_HS_DM: TP1.1, U1.16 (USB_DM)
- new net USB_HS_DP: TP2.1, U1.17 (USB_DP)
- new net VA_RAW: C8.1, FB1.1, U3.5 (OUT)
- no-connect marks 2 -> 40
Other:
- title: (none) -> LoChord
